Commit message: setup referrence in rvis

File: src/rover_description/urdf/rover.urdf (robot description, URDF)
Before this commit: robot rover, 1 links, 0 joints
Links:
- removed link house
- added link base_link; visual box size=0.22 0.15 0.1
- added link referrence; visual mesh filename=file:///home/joshua/Desktop/rover_simulation/src/rover_desc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 scale=0.001 0.001 0.001
Joints:
- added joint referrence: type fixed, parent base_link, child referrence, origin xyz=0 0 0 rpy=0 0 0
