Commit message: simulation can start, not fine tuned yet

File: src/rover_description/urdf/rover.xacro.urdf (robot description, URDF)
Before this commit: robot rover, 10 links, 9 joints
Links:
- added link referrence; visual mesh filename=file:///home/joshua/Desktop/rover_simulation/src/rover_desc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 scale=0.001 0.001 0.001
- link back_left: mass 0.3 -> 0.35
- link back_right: mass 0.3 -> 0.35
- link base_link: mass 5 -> 3
- link bogie_left_back_wheel: mass 0.3 -> 0.35
- link bogie_left_front_wheel: mass 0.3 -> 0.35
- link bogie_right_back_wheel: mass 0.3 -> 0.35
- link bogie_right_front_wheel: mass 0.3 -> 0.35
Joints:
- added joint referrence: type fixed, parent base_link, child referrence, origin xyz=0 0 0 rpy=0 0 0

Commit message: to be squashed with prev commit

File: src/rover_description/urdf/rover.xacro.urdf (robot description, URDF)
Before this commit: robot rover, 11 links, 10 joints
Joints:
- joint bogie_right_joint: type continuous -> revolute

Commit message: fine tuning half way

File: src/rover_description/urdf/rover.xacro.urdf (robot description, URDF)
Before this commit: robot rover, 11 links, 10 joints
Links:
- removed link referrence
- added link rocker_left, mass 0.2; collision cylinder length=0.05 radius=0.015; visual cylinder length=0.05 radius=0.015
- added link rocker_right, mass 0.2; collision cylinder length=0.05 radius=0.015; visual cylinder length=0.05 radius=0.015
Joints:
- removed joint referrence
- added joint rocker_left_joint: type revolute, parent base_link, child rocker_left, origin xyz=-0.075 0.1 0.005 rpy=0 0 0, axis 0.0 1.0 0.0, limit lower=-0.26 upper=0.26 effort=100 velocity=10
- added joint rocker_right_joint: type revolute, parent base_link, child rocker_right, origin xyz=-0.075 -0.1 0.005 rpy=0 0 0, axis 0.0 1.0 0.0, limit lower=-0.26 upper=0.26 effort=100 velocity=10, mimic joint=rocker_left_joint multiplier=-1.0
- joint back_left_joint: origin xyz=-0.17 0.125 -0.115 rpy=0 0 0 -> xyz=-0.095 0.02 -0.12 rpy=0 0 0; parent base_link -> rocker_left
- joint back_right_joint: origin xyz=-0.17 -0.125 -0.115 rpy=0 0 0 -> xyz=-0.095 -0.02 -0.12 rpy=0 0 0; parent base_link -> rocker_right
- joint bogie_left_joint: origin xyz=0.071 0.125 -0.05 rpy=0 0 0 -> xyz=0.145 0.02 -0.055 rpy=0 0 0; parent base_link -> rocker_left
- joint bogie_right_joint: origin xyz=0.071 -0.125 -0.05 rpy=0 0 0 -> xyz=0.145 -0.02 -0.055 rpy=0 0 0; parent base_link -> rocker_right; type revolute -> continuous

Commit message: working simulation

File: src/rover_description/urdf/rover.xacro.urdf (robot description, URDF)
Before this commit: robot rover, 12 links, 11 joints
Links:
- link back_left: mass 0.35 -> 3.7
- link back_right: mass 0.35 -> 3.7
- link base_link: mass 3 -> 2
- link bogie_left_back_wheel: mass 0.35 -> 3.7
- link bogie_left_front_wheel: mass 0.35 -> 3.7
- link bogie_right_back_wheel: mass 0.35 -> 3.7
- link bogie_right_front_wheel: mass 0.35 -> 3.7
Joints:
- joint bogie_left_joint: limit (none) -> lower=1.57 upper=-0.785 effort=100 velocity=10; type continuous -> revolute
- joint bogie_right_joint: limit (none) -> lower=1.57 upper=-0.785 effort=100 velocity=10; type continuous -> revolute
- joint rocker_left_joint: limit lower=-0.26 upper=0.26 effort=100 velocity=10 -> lower=-0.13 upper=0.13 effort=100 velocity=10
- joint rocker_right_joint: limit lower=-0.26 upper=0.26 effort=100 velocity=10 -> lower=-0.13 upper=0.13 effort=100 velocity=10
