Commit message: Added macros to urdf

File: src/rover_description/urdf/effort_rover.xacro.urdf (robot description, URDF)
Before this commit: robot rover, 12 links, 11 joints
Links:
- removed link back_left
- removed link back_right
- removed link bogie_left_back_wheel
- removed link bogie_left_front_wheel
- removed link bogie_right_back_wheel
- removed link bogie_right_front_wheel
- added link back_wheel_left, mass ${wheel_total_mass}; collision cylinder length=0.03 radius=0.057; visual cylinder length=0.03 radius=0.057
- added link back_wheel_right, mass ${wheel_total_mass}; collision cylinder length=0.03 radius=0.057; visual cylinder length=0.03 radius=0.057
- added link bogie_left_wheel_back, mass ${wheel_total_mass}; collision cylinder length=0.03 radius=0.057; visual cylinder length=0.03 radius=0.057
- added link bogie_left_wheel_front, mass ${wheel_total_mass}; collision cylinder length=0.03 radius=0.057; visual cylinder length=0.03 radius=0.057
- added link bogie_right_wheel_back, mass ${wheel_total_mass}; collision cylinder length=0.03 radius=0.057; visual cylinder length=0.03 radius=0.057
- added link bogie_right_wheel_front, mass ${wheel_total_mass}; collision cylinder length=0.03 radius=0.057; visual cylinder length=0.03 radius=0.057
- link bogie_right: geometry collision cylinder length=0.10 radius=0.015; visual cylinder length=0.18 radius=0.015
Joints:
- removed joint back_left_joint
- removed joint back_right_joint
- removed joint bogie_left_back_wheel_joint
- removed joint bogie_left_front_wheel_joint
- removed joint bogie_right_back_wheel_joint
- removed joint bogie_right_front_wheel_joint
- added joint back_wheel_left_joint: type continuous, parent rocker_left, child back_wheel_left, origin xyz=-0.095 0.02 -0.12 rpy=0 0 0, axis 0.0 1.0 0.0
- added joint back_wheel_right_joint: type continuous, parent rocker_right, child back_wheel_right, origin xyz=-0.095 -0.02 -0.12 rpy=0 0 0, axis 0.0 1.0 0.0
- added joint bogie_left_wheel_back_joint: type continuous, parent bogie_left, child bogie_left_wheel_back, origin xyz=-0.08 0 -0.065 rpy=0 0 0, axis 0.0 1.0 0.0
- added joint bogie_left_wheel_front_joint: type continuous, parent bogie_left, child bogie_left_wheel_front, origin xyz=0.08 0 -0.065 rpy=0 0 0, axis 0.0 1.0 0.0
- added joint bogie_right_wheel_back_joint: type continuous, parent bogie_right, child bogie_right_wheel_back, origin xyz=-0.08 0 -0.065 rpy=0 0 0, axis 0.0 1.0 0.0
- added joint bogie_right_wheel_front_joint: type continuous, parent bogie_right, child bogie_right_wheel_front, origin xyz=0.08 0 -0.065 rpy=0 0 0, axis 0.0 1.0 0.0

Commit message: added weight for servos

File: src/rover_description/urdf/effort_rover.xacro.urdf (robot description, URDF)
Before this commit: robot rover, 12 links, 11 joints
Links:
- removed link back_wheel_left
- removed link back_wheel_right
- removed link bogie_left
- removed link bogie_left_wheel_back
- removed link bogie_left_wheel_front
- removed link bogie_right
- removed link bogie_right_wheel_back
- removed link bogie_right_wheel_front
- removed link rocker_left
- removed link rocker_right
Joints:
- removed joint back_wheel_left_joint
- removed joint back_wheel_right_joint
- added joint back_left_wheel_joint: type continuous, parent rocker_left, child back_left_wheel, origin xyz=-0.095 0.02 -0.12 rpy=0 0 0, axis 0.0 1.0 0.0
- added joint back_right_wheel_joint: type continuous, parent rocker_right, child back_right_wheel, origin xyz=-0.095 -0.02 -0.12 rpy=0 0 0, axis 0.0 1.0 0.0
- added joint servo1_joint: type fixed, parent bogie_left, child servo1, origin xyz=0.08 0 0 rpy=0 0 0
- added joint servo2_joint: type fixed, parent bogie_right, child servo2, origin xyz=0.08 0 0 rpy=0 0 0
- added joint servo3_joint: type fixed, parent bogie_left, child servo3, origin xyz=-0.08 0 0 rpy=0 0 0
- added joint servo4_joint: type fixed, parent bogie_right, child servo4, origin xyz=-0.08 0 0 rpy=0 0 0
- added joint servo5_joint: type fixed, parent base_link, child servo5, origin xyz=-0.17 0.14 -0.055 rpy=0 0 0
- added joint servo6_joint: type fixed, parent base_link, child servo6, origin xyz=-0.17 -0.14 -0.055 rpy=0 0 0

Commit message: updated some innertia, not all inertia updated yet

File: src/rover_description/urdf/effort_rover.xacro.urdf (robot description, URDF)
Before this commit: robot rover, 2 links, 17 joints
Links:
- link base_link: mass 2 -> ${mass}

Commit message: completed

File: src/rover_description/urdf/effort_rover.xacro.urdf (robot description, URDF)
Before this commit: robot rover, 2 links, 17 joints
Links:
- link base_link: mass ${mass} -> ${body_mass}
Joints:
- joint servo5_joint: origin xyz=-0.17 0.14 -0.055 rpy=0 0 0 -> xyz=-0.17 0.12 -0.055 rpy=0 0 0
- joint servo6_joint: origin xyz=-0.17 -0.14 -0.055 rpy=0 0 0 -> xyz=-0.17 -0.12 -0.055 rpy=0 0 0

Commit message: added velocity limits to wheels

File: src/rover_description/urdf/effort_rover.xacro.urdf (robot description, URDF)
Before this commit: robot rover, 2 links, 17 joints
Joints:
- joint back_left_wheel_joint: limit (none) -> effort=0.8 velocity=${velocity_limit}
- joint back_right_wheel_joint: limit (none) -> effort=0.8 velocity=${velocity_limit}
- joint bogie_left_wheel_back_joint: limit (none) -> effort=0.8 velocity=${velocity_limit}
- joint bogie_left_wheel_front_joint: limit (none) -> effort=0.8 velocity=${velocity_limit}
- joint bogie_right_wheel_back_joint: limit (none) -> effort=0.8 velocity=${velocity_limit}
- joint bogie_right_wheel_front_joint: limit (none) -> effort=0.8 velocity=${velocity_limit}

Commit message: changed max angle of bogie

File: src/rover_description/urdf/effort_rover.xacro.urdf (robot description, URDF)
Before this commit: robot rover, 2 links, 17 joints
Joints:
- joint bogie_left_joint: limit lower=1.57 upper=-0.436332 effort=100 velocity=10 -> lower=1.57 upper=-0.523599 effort=100 velocity=10
- joint bogie_right_joint: limit lower=1.57 upper=-0.436332 effort=100 velocity=10 -> lower=1.57 upper=-0.523599 effort=100 velocity=10

Commit message: updated to take into acc servo weight

File: src/rover_description/urdf/effort_rover.xacro.urdf (robot description, URDF)
Before this commit: robot rover, 2 links, 17 joints
Links:
- added link referrence; visual mesh filename=file:///home/joshua/Desktop/rover_simulation/src/rover_desc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 scale=0.001 0.001 0.001
Joints:
- added joint referrence: type fixed, parent base_link, child referrence, origin xyz=0 0 0 rpy=0 0 0
- joint back_left_wheel_joint: origin xyz=${rocker_to_back_wheel} 0.02 -0.12 rpy=0 0 0 -> xyz=${rocker_to_back_wheel} -0.02 -0.12 rpy=0 0 0
- joint servo1_joint: origin xyz=0.08 0 0 rpy=0 0 0 -> xyz=${bogie_length/2} 0 0 rpy=0 0 0
- joint servo2_joint: origin xyz=0.08 0 0 rpy=0 0 0 -> xyz=${bogie_length/2} 0 0 rpy=0 0 0
- joint servo3_joint: origin xyz=-0.08 0 0 rpy=0 0 0 -> xyz=-${bogie_length/2} 0 0 rpy=0 0 0
- joint servo4_joint: origin xyz=-0.08 0 0 rpy=0 0 0 -> xyz=-${bogie_length/2} 0 0 rpy=0 0 0
- joint servo5_joint: origin xyz=-0.17 0.12 -0.055 rpy=0 0 0 -> xyz=-0.20 0.12 -0.055 rpy=0 0 0
- joint servo6_joint: origin xyz=-0.17 -0.12 -0.055 rpy=0 0 0 -> xyz=-0.20 -0.12 -0.055 rpy=0 0 0

Commit message: made robot wheelbase equal

File: src/rover_description/urdf/effort_rover.xacro.urdf (robot description, URDF)
Before this commit: robot rover, 3 links, 18 joints
Links:
- removed link referrence
Joints:
- removed joint referrence
- joint servo5_joint: origin xyz=-0.20 0.12 -0.055 rpy=0 0 0 -> xyz=${rocker_to_back_wheel} 0.12 -0.055 rpy=0 0 0
- joint servo6_joint: origin xyz=-0.20 -0.12 -0.055 rpy=0 0 0 -> xyz=${rocker_to_back_wheel} -0.12 -0.055 rpy=0 0 0
