Commit message: Simulation that can climb stairs

File: src/rover_description/urdf/backup/backup.urdf (robot description, URDF)
Before this commit: robot rover, 9 links, 8 joints
Links:
- added link referrence; visual mesh filename=file:///home/joshua/Desktop/rover_simulation/src/rover_desc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 scale=0.001 0.001 0.001
Joints:
- added joint referrence: type fixed, parent base_link, child referrence, origin xyz=0 0 0 rpy=0 0 0

File: src/rover_description/urdf/effort_rover.xacro.urdf (robot description, URDF)
Before this commit: robot rover, 2 links, 17 joints
Joints:
- joint back_left_wheel_joint: limit effort=0.8 velocity=${velocity_limit} -> effort=100 velocity=${velocity_limit}; origin xyz=-0.095 0.02 -0.12 rpy=0 0 0 -> xyz=${rocker_to_back_wheel} 0.02 -0.12 rpy=0 0 0
- joint back_right_wheel_joint: limit effort=0.8 velocity=${velocity_limit} -> effort=100 velocity=${velocity_limit}; origin xyz=-0.095 -0.02 -0.12 rpy=0 0 0 -> xyz=${rocker_to_back_wheel} -0.02 -0.12 rpy=0 0 0
- joint bogie_left_joint: limit lower=1.57 upper=-0.785 effort=100 velocity=10 -> lower=1.57 upper=-0.436332 effort=100 velocity=10; origin xyz=0.145 0.02 -0.055 rpy=0 0 0 -> xyz=${rocker_to_bogie} 0.02 -0.055 rpy=0 0 0
- joint bogie_left_wheel_back_joint: limit effort=0.8 velocity=${velocity_limit} -> effort=100 velocity=${velocity_limit}; origin xyz=-0.08 0 -0.065 rpy=0 0 0 -> xyz=-${bogie_length/2} 0 -0.065 rpy=0 0 0
- joint bogie_left_wheel_front_joint: limit effort=0.8 velocity=${velocity_limit} -> effort=100 velocity=${velocity_limit}; origin xyz=0.08 0 -0.065 rpy=0 0 0 -> xyz=${bogie_length/2} 0 -0.065 rpy=0 0 0
- joint bogie_right_joint: limit lower=1.57 upper=-0.785 effort=100 velocity=10 -> lower=1.57 upper=-0.436332 effort=100 velocity=10; origin xyz=0.145 -0.02 -0.055 rpy=0 0 0 -> xyz=${rocker_to_bogie} -0.02 -0.055 rpy=0 0 0
- joint bogie_right_wheel_back_joint: limit effort=0.8 velocity=${velocity_limit} -> effort=100 velocity=${velocity_limit}; origin xyz=-0.08 0 -0.065 rpy=0 0 0 -> xyz=-${bogie_length/2} 0 -0.065 rpy=0 0 0
- joint bogie_right_wheel_front_joint: limit effort=0.8 velocity=${velocity_limit} -> effort=100 velocity=${velocity_limit}; origin xyz=0.08 0 -0.065 rpy=0 0 0 -> xyz=${bogie_length/2} 0 -0.065 rpy=0 0 0
